File: eagle/automation-v2.brd (EAGLE design)
At the start: 109.5 x 67 mm, 104 parts, among them IC1 MEGA48/88/168-AU, IC2 DS2482-100S, IC3 DS2482-100S, IC4 78L33, IC6 TPS56X200, K1 SRD-05VDC-SL-C, K2 SRD-05VDC-SL-C, K3 SRD-05VDC-SL-C, K4 SRD-05VDC-SL-C, Q1 BSS123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

Commit message: strong 1w pullup added
Parts:
- added Q5, Q6: BSS84, transistor-small-signal:SOT23
- moved C7 0.95 mm to (15.6, 50.8), turned to 270 degrees
Connections:
- net N$1 renamed SDA
- net N$2 renamed SCL
- new net N$21: IC3.6, Q5.1
- new net N$65: IC2.6, Q6.1
- net N$30: now also Q5.3
- net N$60: now also Q6.3
- net VDD: now also Q5.2, Q6.2
Routing:
- net VDD: track 69.3 -> 84.3 mm, vias 3 -> 2
- net N$21: track 0.00 -> 7.84 mm, vias 0 -> 1
- net N$65: track 0.00 -> 7.39 mm, vias 0 -> 1
- net N$60: track 8.41 -> 13.2 mm
- net N$30: track 8.41 -> 13.2 mm
- net SDA: track 52.2 -> 48.9 mm
- net GND: vias 43 -> 44
