File: eagle/automation-v3.sch (EAGLE design)
At the start: 106 parts, among them IC1 MEGA48/88/168-AU, IC2 DS2482-100S, IC3 DS2482-100S, IC4 78L33, IC6 TPS56X200, K1 SRD-05VDC-SL-C, K2 SRD-05VDC-SL-C, K3 SRD-05VDC-SL-C, K4 SRD-05VDC-SL-C, Q1 BSS123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

Commit message: Updated resistor values
Parts:
- IC1: value MEGA48/88/168-AU -> ATmega328P-AU
- IC5: value (none) -> MCP1702T-33
- R1, R2: value (none) -> 150
- R12, R30: value (none) -> 150K 1%
- R15, R16, R17, R19, R20, R25, R26, R3, R4, R9: value (none) -> 10K
- R18, R21, R24, R27: value (none) -> 3.6K
- R22, R23: value (none) -> 390
- R31, R34: value (none) -> 30K 1%
- R36, R37, R38, R39: value (none) -> 120
- R5: value (none) -> 51K 1%
- R6, R7: value (none) -> 4.7K
Other:
- note added: "R11 62K || 470K"
